File: HW2/new_schematic.sch (EAGLE design)
At the start: 2 parts

Commit message: version_1
Parts:
- removed LED1: (no value), led:LED3MM
- removed R1: (no value), resistor:R-US_0207/10
- added 10K, 330: (no value), new_library:R-US_0207/10
- added C1, C2, C3, C4, C5, C6: (no value), new_library:10UF-25V-20%(PTH)KIT
- added G_LED, R_LED: (no value), new_library:LED3MM
- added J1: (no value), new_library:M05NO_SILK
- added R2: 330, new_library:R-US_0207/10
- added R4: 10K, new_library:R-US_0207/10
- added S1, S2: (no value), new_library:MS243
- added S3: (no value), switch:M251
- added U$1: PIC32, new_library:PIC32
- added U$9: MCP1702, new_library:MCP1702
- added X1: HC49-HC49-3L, new_library:HC49-HC49-3L
- added X2: MINI-USB-32005-201, con-cypressindustries:MINI-USB-32005-201
Connections:
- new net +3V3: C1.+, C2.+, C3.+, C4.+, J1.3, R4.1, R_LED.A, U$1.3.3, U$1.P$28, U$1.VDD, U$9.VOUT
- new net GND: 10K.2, 330.1, C2.-, C3.-, C4.-, C5.-, C6.-, J1.2, R2.1, S1.P, S2.P, U$1.P$27, U$1.VSS, U$1.VSS19, X1.2
- new net N$1: U$1.USBID, X2.2
- new net N$10: C5.+, U$1.VCAP
- new net N$11: 330.2, G_LED.C
- new net N$12: G_LED.A, U$1.RA4
- new net N$13: S3.S, X2.5
- new net N$14: C6.+, S3.P, U$1.VBUS, U$9.VIN
- new net N$15: U$1.D-, X2.4
- new net N$16: U$1.D+, X2.3
- new net N$2: J1.4, U$1.PGD1
- new net N$3: J1.5, U$1.PGC1
- new net N$4: U$1.OSC1, X1.1
- new net N$5: U$1.OSC2, X1.3
- new net N$6: 10K.1, S1.S, U$1.RB4
- new net N$7: C1.-, U$9.GND, X2.1
- new net N$8: R2.2, R_LED.C
- new net N$9: J1.1, R4.2, S2.S, U$1.!MCLR

Commit message: 123
Parts:
- removed S1, S2: (no value), new_library:MS243
- removed S3: (no value), switch:M251
- removed X2: MINI-USB-32005-201, con-cypressindustries:MINI-USB-32005-201
- added J2, J3: (no value), new_library:M08
- added U$2: MINI_USB, new_library:MINI_USB
- added U$3: SLIDE_SWITCH, new_library:SLIDE_SWITCH
- added U$4, U$5: PUSH_BUTTON, new_library:PUSH_BUTTON
- C1, C2, C3, C4, C5: value (none) -> 0.1uF; device new_library:10UF-25V-20%(PTH)KIT -> new_library:C-US025-025X050
- C6: value (none) -> 10uF; device new_library:10UF-25V-20%(PTH)KIT -> new_library:CPOL-US150CLZ-0810
Connections:
- new net N$19: J2.1, U$1.P$2
- new net N$20: J2.2, U$1.P$3
- new net N$21: J2.3, U$1.P$6
- new net N$22: J2.4, U$1.P$7
- new net N$23: J3.1, U$1.P$26
- new net N$24: J3.2, U$1.P$25
- new net N$25: J3.3, U$1.P$24
- new net N$26: J3.4, U$1.P$18
- new net N$27: J3.5, U$1.P$17
- new net N$28: J3.6, U$1.P$16
- net +3V3: now also C1.1, C2.1, C3.1, C4.1, J2.7; no longer C1.+, C2.+, C3.+, C4.+
- net GND: now also C1.2, C3.2, C4.2, C5.2, J2.8, J3.8, U$4.2, U$5.1; no longer C2.-, C3.-, C4.-, C5.-, S1.P, S2.P
- net N$1: now also U$2.2.ID; no longer X2.2
- net N$10: now also C6.+; no longer C5.+
- net N$12: now also J2.6
- net N$13: now also U$2.5.VBUS, U$3.2; no longer S3.S, X2.5
- net N$14: now also C5.1, J3.7, U$3.1; no longer C6.+, S3.P
- net N$15: now also U$2.4.D-; no longer X2.4
- net N$16: now also U$2.3.D+; no longer X2.3
- net N$6: now also J2.5, U$5.2; no longer S1.S
- net N$7: now also C2.2, U$2.1.GND; no longer C1.-, X2.1
- net N$9: now also U$4.1; no longer S2.S
Other:
- moved on the sheet: C6
